File: TYPING-TRAINER-V4/TYPING-TRAINER-V4.kicad_sch (KiCad schematic)
At the start: 57 parts, among them J1 Conn_01x20_Pin, J2 Conn_01x02_Pin, M1 Motor_DC, M2 Motor_DC, M3 Motor_DC, M4 Motor_DC, M5 Motor_DC, M6 Motor_DC, M7 Motor_DC, M8 Motor_DC, SW1 SW_DIP_x01, SW10 SW_DIP_x01, SW11 SW_DIP_x01, SW12 SW_DIP_x01, SW13 SW_DIP_x01, SW14 SW_DIP_x01, SW15 SW_DIP_x01, SW16 SW_DIP_x01, SW17 SW_DIP_x01, SW18 SW_DIP_x01, SW19 SW_DIP_x01, SW2 SW_DIP_x01, SW20 SW_DIP_x01, SW21 SW_DIP_x01, SW22 SW_DIP_x01, SW23 SW_DIP_x01, SW24 SW_DIP_x01, SW25 SW_DIP_x02b, SW26 SW_DIP_x02b, SW3 SW_DIP_x01, SW4 SW_DIP_x01, SW5 SW_DIP_x01, SW6 SW_DIP_x01, SW7 SW_DIP_x01, SW8 SW_DIP_x01, SW9 SW_DIP_x01, U2 MCP23017_SP

Commit message: 3rd commit
Parts:
- D4: value LED -> LED 5mm
- J1: value Conn_01x20_Pin -> 20pin PInSocket
- J2: value Conn_01x02_Pin -> 2pin PinSocket
- R1, R10, R11, R2, R3, R4, R5, R6, R7, R8: value R -> 10k
- R9: value R -> 330
- SW1, SW10, SW11, SW12, SW13, SW14, SW15, SW16, SW17, SW18, SW19, SW2, SW20, SW21, SW22, SW23, SW24, SW3, SW4, SW5, SW6, SW7, SW8, SW9: value SW_DIP_x01 -> CherryMX Switch
- SW25, SW26: value SW_DIP_x02b -> Button Switch
- U2: value MCP23017_SP -> MCP23017
Changed lines of the file:
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@@
 		(on_board yes)
 		(dnp no)
-		(fields_autoplaced yes)
 		(property "Reference" "R6"
 			(at 210.82 126.9999 0)
@@
 			)
 		)
-		(property "Value" "R"
-			(at 210.82 129.5399 0)
+		(property "Value" "10k"
+			(at 209.804 129.54 0)
 			(effects
 				(font
@@
 			)
 		)
-		(property "Value" "SW_DIP_x01"
+		(property "Value" "CherryMX Switch"
 			(at 119.38 83.82 0)
 			(effects
@@
 			)
 		)
-		(property "Value" "SW_DIP_x01"
+		(property "Value" "CherryMX Switch"
 			(at 160.02 83.82 0)
 			(effects
@@
 			)
 		)
-		(property "Value" "SW_DIP_x01"
+		(property "Value" "CherryMX Switch"
 			(at 38.1 60.96 0)
 			(effects
@@
 			)
 		)
-		(property "Value" "SW_DIP_x01"
+		(property "Value" "CherryMX Switch"
 			(at 139.7 39.37 0)
 			(effects
@@
 			)
 		)
-		(property "Value" "SW_DIP_x01"
+		(property "Value" "CherryMX Switch"
 			(at 180.34 83.82 0)
 			(effects
@@
 			)
 		)
-		(property "Value" "SW_DIP_x01"
+		(property "Value" "CherryMX Switch"
 			(at 99.06 39.37 0)
 			(effects
@@
 			)
 		)
-		(property "Value" "SW_DIP_x01"
+		(property "Value" "CherryMX Switch"
 			(at 160.02 39.37 0)
 			(effects
@@
 		(on_board yes)
 		(dnp no)
-		(fields_autoplaced yes)
 		(property "Reference" "R2"
 			(at 185.42 126.9999 0)
@@
 			)
 		)
-		(property "Value" "R"
-			(at 185.42 129.5399 0)
+		(property "Value" "10k"
+			(at 184.404 129.54 0)
 			(effects
 				(font
@@
 			)
 		)
-		(property "Value" "SW_DIP_x01"
+		(property "Value" "CherryMX Switch"
 			(at 139.7 60.96 0)
 			(effects
@@
 			)
 		)
-		(property "Value" "MCP23017_SP"
+		(property "Value" "MCP23017"
 			(at 305.7241 59.69 0)
 			(effects
@@
 			)
 		)
-		(property "Value" "SW_DIP_x01"
+		(property "Value" "CherryMX Switch"
 			(at 78.74 60.96 0)
 			(effects
@@
 			)
 		)
-		(property "Value" "Conn_01x02_Pin"
+		(property "Value" "2pin PinSocket"
 			(at 361.95 167.6399 0)
 			(effects
@@
 			)
 		)
-		(property "Value" "Conn_01x20_Pin"
+		(property "Value" "20pin PInSocket"
 			(at 242.57 27.94 90)
 			(effects
@@
 			)
 		)
-		(property "Value" "SW_DIP_x01"
+		(property "Value" "CherryMX Switch"
 			(at 160.02 60.96 0)
 			(effects
@@
 		(on_board yes)
 		(dnp no)
-		(fields_autoplaced yes)
 		(property "Reference" "R8"
 			(at 223.52 126.9999 0)
@@
 			)
 		)
-		(property "Value" "R"
-			(at 223.52 129.5399 0)
+		(property "Value" "10k"
+			(at 222.504 129.54 0)
 			(effects
 				(font
@@
 			)
 		)
-		(property "Value" "R"
+		(property "Value" "10k"
 			(at 261.62 48.2599 0)
 			(effects
@@
 			)
 		)
-		(property "Value" "SW_DIP_x01"
+		(property "Value" "CherryMX Switch"
 			(at 119.38 60.96 0)
 			(effects
@@
 			)
 		)
-		(property "Value" "SW_DIP_x02b"
+		(property "Value" "Button Switch"
 			(at 265.43 64.7699 90)
 			(effects
@@
 			)
 		)
-		(property "Value" "SW_DIP_x01"
+		(property "Value" "CherryMX Switch"
 			(at 58.42 60.96 0)
 			(effects
@@
 		(on_board yes)
 		(dnp no)
-		(fields_autoplaced yes)
 		(property "Reference" "R1"
 			(at 179.07 126.9999 0)
@@
 			)
 		)
-		(property "Value" "R"
-			(at 179.07 129.5399 0)
+		(property "Value" "10k"
+			(at 178.054 129.54 0)
 			(effects
 				(font
@@
 			)
 		)
-		(property "Value" "R"
+		(property "Value" "10k"
 			(at 270.51 48.2599 0)
 			(effects
@@
 			)
 		)
-		(property "Value" "SW_DIP_x01"
+		(property "Value" "CherryMX Switch"
 			(at 119.38 39.37 0)
 			(effects
@@
 		(on_board yes)
 		(dnp no)
-		(fields_autoplaced yes)
 		(property "Reference" "SW26"
-			(at 281.94 74.9299 90)
+			(at 259.334 75.184 90)
 			(effects
 				(font
@@
 			)
 		)
-		(property "Value" "SW_DIP_x02b"
-			(at 281.94 77.4699 90)
+		(property "Value" "Button Switch"
+			(at 259.334 77.724 90)
 			(effects
 				(font
@@
 			)
 		)
-		(property "Value" "SW_DIP_x01"
+		(property "Value" "CherryMX Switch"
 			(at 38.1 83.82 0)
 			(effects
@@
 			)
 		)
-		(property "Value" "SW_DIP_x01"
+		(property "Value" "CherryMX Switch"
 			(at 58.42 83.82 0)
 			(effects
@@
 		(on_board yes)
 		(dnp no)
-		(fields_autoplaced yes)
 		(property "Reference" "R4"
 			(at 198.12 126.9999 0)
@@
 			)
 		)
-		(property "Value" "R"
-			(at 198.12 129.5399 0)
+		(property "Value" "10k"
+			(at 197.104 129.54 0)
 			(effects
 				(font
@@
 			)
 		)
-		(property "Value" "SW_DIP_x01"
+		(property "Value" "CherryMX Switch"
 			(at 78.74 39.37 0)
 			(effects
@@
 			)
 		)
-		(property "Value" "SW_DIP_x01"
+		(property "Value" "CherryMX Switch"
 			(at 58.42 39.37 0)
 			(effects
@@
 			)
 		)
-		(property "Value" "SW_DIP_x01"
+		(property "Value" "CherryMX Switch"
 			(at 38.1 39.37 0)
 			(effects
@@
 			)
 		)
-		(property "Value" "SW_DIP_x01"
+		(property "Value" "CherryMX Switch"
 			(at 180.34 60.96 0)
 			(effects
@@
 			)
 		)
-		(property "Value" "SW_DIP_x01"
+		(property "Value" "CherryMX Switch"
 			(at 99.06 60.96 0)
 			(effects
@@
 			)
 		)
-		(property "Value" "R"
+		(property "Value" "330"
 			(at 248.92 99.0599 0)
 			(effects
@@
 		(on_board yes)
 		(dnp no)
-		(fields_autoplaced yes)
 		(property "Reference" "R3"
 			(at 191.77 126.9999 0)
@@
 			)
 		)
-		(property "Value" "R"
-			(at 191.77 129.5399 0)
+		(property "Value" "10k"
+			(at 190.754 129.54 0)
 			(effects
 				(font
@@
 			)
 		)
-		(property "Value" "SW_DIP_x01"
+		(property "Value" "CherryMX Switch"
 			(at 99.06 83.82 0)
 			(effects
@@
 			)
 		)
-		(property "Value" "SW_DIP_x01"
+		(property "Value" "CherryMX Switch"
 			(at 78.74 83.82 0)
 			(effects
@@
 		(on_board yes)
 		(dnp no)
-		(fields_autoplaced yes)
 		(property "Reference" "R5"
 			(at 204.47 126.9999 0)
@@
 			)
 		)
-		(property "Value" "R"
-			(at 204.47 129.5399 0)
+		(property "Value" "10k"
+			(at 203.454 129.54 0)
 			(effects
 				(font
@@
 		(on_board yes)
 		(dnp no)
-		(fields_autoplaced yes)
 		(property "Reference" "R7"
 			(at 217.17 126.9999 0)
@@
 			)
 		)
-		(property "Value" "R"
-			(at 217.17 129.5399 0)
+		(property "Value" "10k"
+			(at 216.154 129.54 0)
 			(effects
 				(font
@@
 			)
 		)
-		(property "Value" "SW_DIP_x01"
+		(property "Value" "CherryMX Switch"
 			(at 139.7 83.82 0)
 			(effects
@@
 			)
 		)
-		(property "Value" "SW_DIP_x01"
+		(property "Value" "CherryMX Switch"
 			(at 180.34 39.37 0)
 			(effects
@@
 			)
 		)
-		(property "Value" "LED"
+		(property "Value" "LED 5mm"
 			(at 250.19 112.0774 90)
 			(effects
